Commit message: Complete the design and add a config file

File: urdf/robo_dif.xacro (robot description, xacro)
@@ -2,6 +2,7 @@
 <!-- robot description-->
 <robot name="robo_ dif" xmlns:xacro="http://www.ros.org/wiki/xacro">
-  <!--chassis-->
+  <!--base link-->
   <link name="base_link">
+    <!--chassis-->
     <visual>
       <origin rpy="0 0 0" xyz="0 0 0"/>
@@ -9,4 +10,11 @@
         <box size="0.5 0.3 0.07"/>
       </geometry>
+    </visual>
+    <!--caster front-->
+    <visual>
+      <origin rpy=" 0 0 0" xyz="0.2 0 -0.05"/>
+        <geometry>
+          <sphere radius="0.05"/>
+        </geometry>
     </visual>
   </link>

Commit message: add collisions

File: urdf/robo_dif.xacro (robot description, xacro)
@@ -4,5 +4,5 @@
   <!--base link-->
   <link name="base_link">
-    <!--chassis-->
+    <!--chassis visual-->
     <visual>
       <origin rpy="0 0 0" xyz="0 0 0"/>
@@ -11,5 +11,11 @@
       </geometry>
     </visual>
-    <!--caster front-->
+    <!--chassis collision-->
+    <collision>
+      <geometry>
+        <box size="0.5 0.3 0.07"/>
+      </geometry>
+    </collision>
+    <!--caster front visual-->
     <visual>
       <origin rpy=" 0 0 0" xyz="0.2 0 -0.05"/>
@@ -18,7 +24,25 @@
         </geometry>
     </visual>
+    <!--caster front collision-->
+    <collision>
+      <origin rpy=" 0 0 0" xyz="0.35 0 -0.05"/>
+      <geometry>
+        <sphere radius="0.05"/>
+      </geometry>
+      <surface>
+        <friction>
+          <ode>
+            <mu>0</mu>
+            <mu2>0</mu2>
+            <slip1>1.0</slip1>
+            <slip2>1.0</slip2>
+          </ode>
+        </friction>
+      </surface>
+    </collision>
   </link>
   <!--left wheel-->
   <link name="lwheel">
+    <!--left wheel visual-->
     <visual>
       <origin rpy="0 1.5707 1.5707" xyz="0 0 0"/>
@@ -27,7 +51,14 @@
       </geometry>
     </visual>
+    <!--left wheel collision-->
+    <collision>
+      <geometry>
+        <cylinder length="0.04" radius="0.1"/>
+      </geometry>
+    </collision>
   </link>
   <!--right wheel-->
   <link name="rwheel">
+    <!--right wheel visual-->
     <visual>
       <origin rpy="0 1.5707 1.5707" xyz="0 0 0"/>
@@ -36,4 +67,10 @@
       </geometry>
     </visual>
+    <!--right wheel collision-->
+    <collision>
+      <geometry>
+        <cylinder length="0.04" radius="0.1"/>
+      </geometry>
+    </collision>
   </link>
   <!--joint for left wheel-->

Commit message: add inertial

File: urdf/robo_dif.xacro (robot description, xacro)
@@ -17,4 +17,10 @@
       </geometry>
     </collision>
+    <!--chassis inertial-->
+    <inertial>
+      <mass value="5"/>
+      <origin rpy="0 0 0" xyz="0 0 0.1"/>
+      <inertia ixx="0.0395416666667" ixy="0" ixz="0" iyy="0.106208333333" iyz="0" izz="0.106208333333"/>
+    </inertial>
     <!--caster front visual-->
     <visual>
@@ -57,4 +63,10 @@
       </geometry>
     </collision>
+    <!--left wheel inertial-->
+    <inertial>
+      <mass value="0.2"/>
+      <origin rpy="0 1.5707 1.5707" xyz="0 0 0"/>
+      <inertia ixx="0.00052666666" ixy="0" ixz="0" iyy="0.00052666666" iyz="0" izz="0.001"/>
+    </inertial>
   </link>
   <!--right wheel-->
@@ -73,4 +85,10 @@
       </geometry>
     </collision>
+    <!--right wheel inertial-->
+    <inertial>
+      <mass value="0.2"/>
+      <origin rpy="0 1.5707 1.5707" xyz="0 0 0"/>
+      <inertia ixx="0.00052666666" ixy="0" ixz="0" iyy="0.00052666666" iyz="0" izz="0.001"/>
+    </inertial>
   </link>
   <!--joint for left wheel-->

Commit message: gazebo simulation and solve problems

File: urdf/robo_dif.xacro (robot description, xacro)
@@ -4,4 +4,6 @@
   <!--base link-->
   <link name="base_link">
+    <!--base link pose-->
+    <pose>0 0 0.1 0 0 0</pose>
     <!--chassis visual-->
     <visual>
@@ -59,4 +61,5 @@
     <!--left wheel collision-->
     <collision>
+      <origin rpy="0 1.5707 1.5707" xyz="0 0 0"/>
       <geometry>
         <cylinder length="0.04" radius="0.1"/>
@@ -81,4 +84,5 @@
     <!--right wheel collision-->
     <collision>
+      <origin rpy="0 1.5707 1.5707" xyz="0 0 0"/>
       <geometry>
         <cylinder length="0.04" radius="0.1"/>

Commit message: sensor laser and macro file

File: urdf/robo_dif.xacro (robot description, xacro)
@@ -1,5 +1,8 @@
 <?xml version="1.0"?>
-<!-- robot description-->
+<!--robot description-->
 <robot name="robo_ dif" xmlns:xacro="http://www.ros.org/wiki/xacro">
+  <!-- ############################# INCLUDES ##########################  -->
+  <xacro:include filename="$(find urdf_teste)/urdf/macro.xacro" />
+  <!-- ############################# LINKS #############################  -->
   <!--base link-->
   <link name="base_link">
@@ -96,4 +99,28 @@
     </inertial>
   </link>
+  <!--sensor laser-->
+  <link name="sensor_laser">
+    <!--sensor laser visual-->
+    <visual>
+      <origin xyz="0 0 0" rpy="0 0 0" />
+      <geometry>
+        <cylinder radius="0.05" length="0.1"/>
+      </geometry>
+    </visual>
+    <!--sensor laser collision-->
+    <collision>
+      <origin xyz="0 0 0" rpy="0 0 0"/>
+      <geometry>
+        <cylinder radius="0.05" length="0.1"/>
+      </geometry>
+    </collision>
+    <!--sensor laser inertial-->
+    <inertial>
+      <origin xyz="0 0 0" rpy="0 0 0" />
+      <mass value="1" />
+      <xacro:cylinder_inertia mass="1" r="0.05" l="0.1" />
+    </inertial>
+  </link>
+  <!-- ############################# JOINTS #############################  -->
   <!--joint for left wheel-->
   <joint name="joint_left_wheel" type="continuous">
@@ -114,3 +141,58 @@
     <joint_properties damping="1.0" friction="1.0" />
   </joint>
+  <!--joint for sensor laser-->
+  <joint name="joint_sensor_laser" type="fixed">
+    <origin xyz="0.15 0 0.05" rpy="0 0 0"/>
+    <parent link="base_link"/>
+    <child link="sensor_laser"/>
+  </joint>
+  <!-- ############################# PLUGINS #############################  -->
+  <!--gazebo diferential drive plugin-->
+  <gazebo>
+    <plugin filename="libgazebo_ros_diff_drive.so" name="differential_drive_controller">
+      <alwaysOn>true</alwaysOn>
+      <updateRate>20</updateRate>
+      <leftJoint>joint_left_wheel</leftJoint>
+      <rightJoint>joint_right_wheel</rightJoint>
+      <wheelSeparation>0.4</wheelSeparation>
+      <wheelDiameter>0.2</wheelDiameter>
+      <torque>0.1</torque>
+      <commandTopic>cmd_vel</commandTopic>
+      <odometryTopic>odom</odometryTopic>
+      <odometryFrame>odom</odometryFrame>
+      <robotBaseFrame>link_chassis</robotBaseFrame>
+    </plugin>
+  </gazebo>
+  <!--gazebo sensor laser plugin-->
+  <gazebo reference="sensor_laser">
+    <sensor type="ray" name="head_hokuyo_sensor">
+      <pose>0 0 0 0 0 0</pose>
+      <visualize>false</visualize>
+      <update_rate>20</update_rate>
+      <ray>
+        <scan>
+          <horizontal>
+            <samples>720</samples>
+            <resolution>1</resolution>
+            <min_angle>-1.570796</min_angle>
+            <max_angle>1.570796</max_angle>
+          </horizontal>
+        </scan>
+        <range>
+          <min>0.10</min>
+          <max>10.0</max>
+          <resolution>0.01</resolution>
+        </range>
+        <noise>
+          <type>gaussian</type>
+          <mean>0.0</mean>
+          <stddev>0.01</stddev>
+        </noise>
+      </ray>
+      <plugin name="gazebo_ros_head_hokuyo_controller" filename="libgazebo_ros_laser.so">
+        <topicName>/robo_dif/laser/scan</topicName>
+        <frameName>sensor_laser</frameName>
+      </plugin>
+    </sensor>
+  </gazebo>
 </robot>

Commit message: depth camera

File: urdf/robo_dif.xacro (robot description, xacro)
@@ -122,4 +122,15 @@
     </inertial>
   </link>
+  <!--depth camera-->
+  <link name="depth_camera">
+    <!--depth camera visual-->
+    <visual>
+      <origin xyz="0 0 0" rpy="0 0 0" />
+      <geometry>
+        <!-- <cylinder radius="0.05" length="0.1"/> -->
+        <box size="0.05 0.05 0.05"/>
+      </geometry>
+    </visual>
+  </link>
   <!-- ############################# JOINTS #############################  -->
   <!--joint for left wheel-->
@@ -146,4 +157,10 @@
     <parent link="base_link"/>
     <child link="sensor_laser"/>
+  </joint>
+  <!--joint for depth camera-->
+  <joint name="joint_depth_camera" type="fixed">
+    <origin xyz="0.15 0 0.13" rpy="0 0 0"/>
+    <parent link="base_link"/>
+    <child link="depth_camera"/>
   </joint>
   <!-- ############################# PLUGINS #############################  -->
@@ -196,3 +213,47 @@
     </sensor>
   </gazebo>
+  <!--gazebo depth camera plugin-->
+  <gazebo reference="depth_camera">
+    <sensor type="depth" name="depth_camera">
+      <always_on>true</always_on>
+      <visualize>true</visualize>
+      <camera>
+          <horizontal_fov>1.047</horizontal_fov>
+          <image>
+              <width>640</width>
+              <height>480</height>
+              <format>R8G8B8</format>
+          </image>
+          <depth_camera>
+          </depth_camera>
+          <clip>
+              <near>0.1</near>
+              <far>100</far>
+          </clip>
+      </camera>
+      <plugin name="camera_controller" filename="libgazebo_ros_openni_kinect.so">
+          <baseline>0.2</baseline>
+          <alwaysOn>true</alwaysOn>
+              <updateRate>10.0</updateRate>
+              <cameraName>depth_camera</cameraName>
+              <frameName>depth_camera</frameName>
+          <imageTopicName>rgb/image_raw</imageTopicName>
+          <depthImageTopicName>depth/image_raw</depthImageTopicName>
+          <pointCloudTopicName>depth/points</pointCloudTopicName>
+          <cameraInfoTopicName>rgb/camera_info</cameraInfoTopicName>
+          <depthImageCameraInfoTopicName>depth/camera_info</depthImageCameraInfoTopicName>
+          <pointCloudCutoff>0.4</pointCloudCutoff>
+              <hackBaseline>0.07</hackBaseline>
+              <distortionK1>0.0</distortionK1>
+              <distortionK2>0.0</distortionK2>
+              <distortionK3>0.0</distortionK3>
+              <distortionT1>0.0</distortionT1>
+              <distortionT2>0.0</distortionT2>
+          <CxPrime>0.0</CxPrime>
+          <Cx>0.0</Cx>
+          <Cy>0.0</Cy>
+          <focalLength>0.0</focalLength>
+          </plugin>
+    </sensor>
+  </gazebo>
 </robot>
